File: Synthesizer/2channelmixer.kicad_sch (KiCad schematic)
At the start: 10 parts

Commit message: Update documentation on learnings
Parts:
- removed R1k: R, symbol Device:R
- added J?: AudioJack2_Ground, symbol Connector:AudioJack2_Ground
- added RV5kohm: R_Potentiometer, symbol Device:R_Potentiometer
Connections:
- net GND: now also J?.G
- net at R100k.2, U?.6: now also RV5kohm.1
- new net: J?.S, J?.T, RV5kohm.2
- no-connect marks 0 -> 1
Changed lines of the file:
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@@
   (junction (at 123.19 57.15) (diameter 0) (color 0 0 0 0)
   )
+  (junction (at 167.64 44.45) (diameter 0) (color 0 0 0 0)
+  )
   (junction (at 143.51 54.61) (diameter 0) (color 0 0 0 0)
   )
@@
   (junction (at 102.87 54.61) (diameter 0) (color 0 0 0 0)
   )
+  (no_connect (at 160.02 54.61))
   (wire (pts (xy 102.87 72.39) (xy 99.06 72.39))
     (stroke (width 0) (type default) (color 0 0 0 0))
@@
     (stroke (width 0) (type default) (color 0 0 0 0))
   )
+  (wire (pts (xy 167.64 44.45) (xy 167.64 45.72))
+    (stroke (width 0) (type default) (color 0 0 0 0))
+  )
   (wire (pts (xy 123.19 72.39) (xy 123.19 57.15))
     (stroke (width 0) (type default) (color 0 0 0 0))
@@
     (stroke (width 0) (type default) (color 0 0 0 0))
   )
+  (wire (pts (xy 156.21 44.45) (xy 167.64 44.45))
+    (stroke (width 0) (type default) (color 0 0 0 0))
+  )
   (wire (pts (xy 102.87 54.61) (xy 105.41 54.61))
     (stroke (width 0) (type default) (color 0 0 0 0))
   )
+  (wire (pts (xy 156.21 50.8) (xy 156.21 44.45))
+    (stroke (width 0) (type default) (color 0 0 0 0))
+  )
   (wire (pts (xy 66.04 36.83) (xy 72.39 36.83))
     (stroke (width 0) (type default) (color 0 0 0 0))
@@
     (stroke (width 0) (type default) (color 0 0 0 0))
   )
-  (wire (pts (xy 147.32 54.61) (xy 143.51 54.61))
+  (wire (pts (xy 167.64 43.18) (xy 167.64 44.45))
+    (stroke (width 0) (type default) (color 0 0 0 0))
+  )
+  (wire (pts (xy 152.4 54.61) (xy 143.51 54.61))
     (stroke (width 0) (type default) (color 0 0 0 0))
   )
@@
   )
   (wire (pts (xy 45.72 54.61) (xy 54.61 54.61))
-    (stroke (width 0) (type default) (color 0 0 0 0))
-  )
-  (wire (pts (xy 154.94 54.61) (xy 160.02 54.61))
     (stroke (width 0) (type default) (color 0 0 0 0))
   )
@@
     )
   )
-  (global_label "Combined output" (shape output) (at 160.02 54.61 0) (fields_autoplaced)
-    (effects (font (size 1.27 1.27)) (justify left))
-    (property "Intersheet References" "${INTERSHEET_REFS}" (id 0) (at 178.7012 54.5306 0)
-      (effects (font (size 1.27 1.27)) (justify left) hide)
-    )
-  )
   (global_label "Wave input 1" (shape input) (at 45.72 33.02 180) (fields_autoplaced)
     (effects (font (size 1.27 1.27)) (justify right))
@@
     )
     (property "Datasheet" "~" (id 3) (at 95.25 72.39 0)
-      (effects (font (size 1.27 1.27)) hide)
-    )
-    (pin "1")
-    (pin "2")
-  )
-  (symbol (lib_id "Device:R") (at 151.13 54.61 90) (unit 1)
-    (in_bom yes) (on_board yes) (fields_autoplaced)
-    (property "Reference" "R1k" (id 0) (at 151.13 48.26 90))
-    (property "Value" "R" (id 1) (at 151.13 50.8 90))
-    (property "Footprint" "" (id 2) (at 151.13 56.388 90)
-      (effects (font (size 1.27 1.27)) hide)
-    )
-    (property "Datasheet" "~" (id 3) (at 151.13 54.61 0)
       (effects (font (size 1.27 1.27)) hide)
     )
@@
     (pin "2")
   )
+  (symbol (lib_id "Connector:AudioJack2_Ground") (at 172.72 43.18 180) (unit 1)
+    (in_bom yes) (on_board yes) (fields_autoplaced)
+    (property "Reference" "J?" (id 0) (at 177.8 42.5449 0)
+      (effects (font (size 1.27 1.27)) (justify right))
+    )
+    (property "Value" "AudioJack2_Ground" (id 1) (at 177.8 45.0849 0)
+      (effects (font (size 1.27 1.27)) (justify right))
+    )
+    (property "Footprint" "" (id 2) (at 172.72 43.18 0)
+      (effects (font (size 1.27 1.27)) hide)
+    )
+    (property "Datasheet" "~" (id 3) (at 172.72 43.18 0)
+      (effects (font (size 1.27 1.27)) hide)
+    )
+    (pin "G")
+    (pin "S")
+    (pin "T")
+  )
   (symbol (lib_id "Device:R") (at 135.89 72.39 90) (unit 1)
     (in_bom yes) (on_board yes) (fields_autoplaced)
@@
     (pin "1")
   )
+  (symbol (lib_id "power:GND") (at 172.72 38.1 180) (unit 1)
+    (in_bom yes) (on_board yes)
+    (property "Reference" "#PWR?" (id 0) (at 172.72 31.75 0)
+      (effects (font (size 1.27 1.27)) hide)
+    )
+    (property "Value" "GND" (id 1) (at 172.72 30.48 90)
+      (effects (font (size 1.27 1.27)) (justify left))
+    )
+    (property "Footprint" "" (id 2) (at 172.72 38.1 0)
+      (effects (font (size 1.27 1.27)) hide)
+    )
+    (property "Datasheet" "" (id 3) (at 172.72 38.1 0)
+      (effects (font (size 1.27 1.27)) hide)
+    )
+    (pin "1")
+  )
+  (symbol (lib_id "Device:R_Potentiometer") (at 156.21 54.61 90) (unit 1)
+    (in_bom yes) (on_board yes)
+    (property "Reference" "RV5kohm" (id 0) (at 154.9399 57.15 0)
+      (effects (font (size 1.27 1.27)) (justify right))
+    )
+    (property "Value" "R_Potentiometer" (id 1) (at 157.4799 57.15 0)
+      (effects (font (size 1.27 1.27)) (justify right))
+    )
+    (property "Footprint" "" (id 2) (at 156.21 54.61 0)
+      (effects (font (size 1.27 1.27)) hide)
+    )
+    (property "Datasheet" "~" (id 3) (at 156.21 54.61 0)
+      (effects (font (size 1.27 1.27)) hide)
+    )
+    (pin "1")
+    (pin "2")
+    (pin "3")
+  )
   (symbol (lib_id "Amplifier_Operational:AD8001AN") (at 130.81 54.61 0) (unit 1)
