File: Synthesizer/miditToCV.kicad_sch (KiCad schematic)
At the start: 11 parts

Commit message: Update documentation on learnings
Parts:
- removed U?: Buck_converter, symbol New_Library:Buck_converter
- added 0.1µF, 0.33µF: C, symbol Device:C
- added U?: LM7805_TO220, Package_TO_SOT_THT:TO-220-3_Vertical, symbol Regulator_Linear:LM7805_TO220
Connections:
- net +12V: now also 0.33µF.2, U?.1 (VI)
- net +5V: now also 0.1µF.2, U?.3 (VO)
- net GND: now also 0.1µF.1, 0.33µF.1, U?.2 (GND)
Other:
- moved on the sheet: 220ohm?, D?, J?
