File: Synthesizer/powerSupply.kicad_sch (KiCad schematic)
At the start: 16 parts

Commit message: Update documentation on learnings
Parts:
- removed 1µF? (x4): C_Polarized, symbol Device:C_Polarized
- added 1µF (x4): C, symbol Device:C
Connections:
- net +12V: now also 1µF.1
- net -12V: now also 1µF.2
- net GND: now also 1µF.1, 1µF.1, 1µF.2, 1µF.2
- net at 4700µF?.2, 4700µF?.2, 4700µF?.2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: now also 1µF.2
- net at 4700µF?.1, 4700µF?.1, 4700µF?.1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: now also 1µF.1
Changed lines of the file:
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@@
   (junction (at 179.07 95.25) (diameter 0) (color 0 0 0 0)
   )
+  (junction (at 157.48 106.68) (diameter 0) (color 0 0 0 0)
+  )
+  (junction (at 157.48 78.74) (diameter 0) (color 0 0 0 0)
+  )
+  (junction (at 138.43 78.74) (diameter 0) (color 0 0 0 0)
+  )
+  (junction (at 100.33 78.74) (diameter 0) (color 0 0 0 0)
+  )
+  (junction (at 190.5 95.25) (diameter 0) (color 0 0 0 0)
+  )
+  (junction (at 138.43 95.25) (diameter 0) (color 0 0 0 0)
+  )
+  (junction (at 170.18 78.74) (diameter 0) (color 0 0 0 0)
+  )
+  (junction (at 190.5 78.74) (diameter 0) (color 0 0 0 0)
+  )
+  (junction (at 100.33 95.25) (diameter 0) (color 0 0 0 0)
+  )
   (junction (at 190.5 106.68) (diameter 0) (color 0 0 0 0)
   )
-  (junction (at 157.48 106.68) (diameter 0) (color 0 0 0 0)
-  )
-  (junction (at 138.43 78.74) (diameter 0) (color 0 0 0 0)
-  )
-  (junction (at 100.33 78.74) (diameter 0) (color 0 0 0 0)
-  )
-  (junction (at 190.5 95.25) (diameter 0) (color 0 0 0 0)
-  )
-  (junction (at 138.43 95.25) (diameter 0) (color 0 0 0 0)
-  )
-  (junction (at 157.48 78.74) (diameter 0) (color 0 0 0 0)
-  )
-  (junction (at 170.18 78.74) (diameter 0) (color 0 0 0 0)
-  )
-  (junction (at 190.5 78.74) (diameter 0) (color 0 0 0 0)
-  )
-  (junction (at 100.33 95.25) (diameter 0) (color 0 0 0 0)
-  )
   (junction (at 119.38 106.68) (diameter 0) (color 0 0 0 0)
   )
@@
     (stroke (width 0) (type default) (color 0 0 0 0))
   )
+  (wire (pts (xy 186.69 106.68) (xy 190.5 106.68))
+    (stroke (width 0) (type default) (color 0 0 0 0))
+  )
+  (wire (pts (xy 93.98 106.68) (xy 100.33 106.68))
+    (stroke (width 0) (type default) (color 0 0 0 0))
+  )
+  (wire (pts (xy 182.88 67.31) (xy 190.5 67.31))
+    (stroke (width 0) (type default) (color 0 0 0 0))
+  )
+  (wire (pts (xy 138.43 106.68) (xy 157.48 106.68))
+    (stroke (width 0) (type default) (color 0 0 0 0))
+  )
+  (wire (pts (xy 179.07 95.25) (xy 179.07 86.36))
+    (stroke (width 0) (type default) (color 0 0 0 0))
+  )
+  (wire (pts (xy 157.48 95.25) (xy 179.07 95.25))
+    (stroke (width 0) (type default) (color 0 0 0 0))
+  )
+  (wire (pts (xy 175.26 67.31) (xy 170.18 67.31))
+    (stroke (width 0) (type default) (color 0 0 0 0))
+  )
+  (wire (pts (xy 186.69 78.74) (xy 190.5 78.74))
+    (stroke (width 0) (type default) (color 0 0 0 0))
+  )
+  (wire (pts (xy 190.5 78.74) (xy 210.82 78.74))
+    (stroke (width 0) (type default) (color 0 0 0 0))
+  )
+  (wire (pts (xy 138.43 95.25) (xy 157.48 95.25))
+    (stroke (width 0) (type default) (color 0 0 0 0))
+  )
+  (wire (pts (xy 190.5 95.25) (xy 190.5 99.06))
+    (stroke (width 0) (type default) (color 0 0 0 0))
+  )
+  (wire (pts (xy 119.38 106.68) (xy 138.43 106.68))
+    (stroke (width 0) (type default) (color 0 0 0 0))
+  )
+  (wire (pts (xy 100.33 86.36) (xy 100.33 95.25))
+    (stroke (width 0) (type default) (color 0 0 0 0))
+  )
+  (wire (pts (xy 190.5 86.36) (xy 190.5 95.25))
+    (stroke (width 0) (type default) (color 0 0 0 0))
+  )
+  (wire (pts (xy 93.98 78.74) (xy 100.33 78.74))
+    (stroke (width 0) (type default) (color 0 0 0 0))
+  )
   (wire (pts (xy 190.5 106.68) (xy 210.82 106.68))
     (stroke (width 0) (type default) (color 0 0 0 0))
   )
-  (wire (pts (xy 93.98 106.68) (xy 100.33 106.68))
-    (stroke (width 0) (type default) (color 0 0 0 0))
-  )
-  (wire (pts (xy 182.88 67.31) (xy 190.5 67.31))
+  (wire (pts (xy 77.47 90.17) (xy 86.36 90.17))
+    (stroke (width 0) (type default) (color 0 0 0 0))
+  )
+  (wire (pts (xy 100.33 78.74) (xy 119.38 78.74))
     (stroke (width 0) (type default) (color 0 0 0 0))
   )
@@
     (stroke (width 0) (type default) (color 0 0 0 0))
   )
-  (wire (pts (xy 179.07 95.25) (xy 179.07 86.36))
-    (stroke (width 0) (type default) (color 0 0 0 0))
-  )
-  (wire (pts (xy 157.48 95.25) (xy 179.07 95.25))
-    (stroke (width 0) (type default) (color 0 0 0 0))
-  )
-  (wire (pts (xy 175.26 67.31) (xy 170.18 67.31))
-    (stroke (width 0) (type default) (color 0 0 0 0))
-  )
-  (wire (pts (xy 186.69 78.74) (xy 190.5 78.74))
-    (stroke (width 0) (type default) (color 0 0 0 0))
-  )
-  (wire (pts (xy 190.5 78.74) (xy 210.82 78.74))
-    (stroke (width 0) (type default) (color 0 0 0 0))
-  )
-  (wire (pts (xy 138.43 95.25) (xy 157.48 95.25))
-    (stroke (width 0) (type default) (color 0 0 0 0))
-  )
-  (wire (pts (xy 190.5 95.25) (xy 190.5 99.06))
-    (stroke (width 0) (type default) (color 0 0 0 0))
-  )
-  (wire (pts (xy 119.38 106.68) (xy 138.43 106.68))
-    (stroke (width 0) (type default) (color 0 0 0 0))
-  )
-  (wire (pts (xy 100.33 86.36) (xy 100.33 95.25))
-    (stroke (width 0) (type default) (color 0 0 0 0))
-  )
-  (wire (pts (xy 190.5 86.36) (xy 190.5 95.25))
-    (stroke (width 0) (type default) (color 0 0 0 0))
-  )
-  (wire (pts (xy 93.98 78.74) (xy 100.33 78.74))
-    (stroke (width 0) (type default) (color 0 0 0 0))
-  )
-  (wire (pts (xy 186.69 106.68) (xy 190.5 106.68))
-    (stroke (width 0) (type default) (color 0 0 0 0))
-  )
-  (wire (pts (xy 77.47 90.17) (xy 86.36 90.17))
-    (stroke (width 0) (type default) (color 0 0 0 0))
-  )
-  (wire (pts (xy 100.33 78.74) (xy 119.38 78.74))
+  (wire (pts (xy 157.48 78.74) (xy 170.18 78.74))
     (stroke (width 0) (type default) (color 0 0 0 0))
   )
@@
   )
   (wire (pts (xy 138.43 78.74) (xy 157.48 78.74))
-    (stroke (width 0) (type default) (color 0 0 0 0))
-  )
-  (wire (pts (xy 157.48 78.74) (xy 170.18 78.74))
-    (stroke (width 0) (type default) (color 0 0 0 0))
-  )
-  (wire (pts (xy 138.43 106.68) (xy 157.48 106.68))
     (stroke (width 0) (type default) (color 0 0 0 0))
   )
@@
   (label "GND" (at 78.74 95.25 0)
     (effects (font (size 1.27 1.27)) (justify left bottom))
-  )
-  (symbol (lib_id "Device:C_Polarized") (at 190.5 82.55 0) (unit 1)
-    (in_bom yes) (on_board yes) (fields_autoplaced)
-    (property "Reference" "1µF?" (id 0) (at 194.31 80.3909 0)
-      (effects (font (size 1.27 1.27)) (justify left))
-    )
-    (property "Value" "C_Polarized" (id 1) (at 194.31 82.9309 0)
-      (effects (font (size 1.27 1.27)) (justify left))
-    )
-    (property "Footprint" "" (id 2) (at 191.4652 86.36 0)
-      (effects (font (size 1.27 1.27)) hide)
-    )
-    (property "Datasheet" "~" (id 3) (at 190.5 82.55 0)
-      (effects (font (size 1.27 1.27)) hide)
-    )
-    (pin "1")
-    (pin "2")
   )
   (symbol (lib_id "Device:C_Polarized") (at 100.33 102.87 0) (unit 1)
@@
     (pin "3")
   )
+  (symbol (lib_id "Device:C") (at 190.5 82.55 0) (unit 1)
+    (in_bom yes) (on_board yes) (fields_autoplaced)
+    (property "Reference" "1µF" (id 0) (at 193.7139 81.2799 0)
+      (effects (font (size 1.27 1.27)) (justify left))
+    )
+    (property "Value" "C" (id 1) (at 193.7139 83.8199 0)
+      (effects (font (size 1.27 1.27)) (justify left))
+    )
+    (property "Footprint" "" (id 2) (at 191.4652 86.36 0)
+      (effects (font (size 1.27 1.27)) hide)
+    )
+    (property "Datasheet" "~" (id 3) (at 190.5 82.55 0)
+      (effects (font (size 1.27 1.27)) hide)
+    )
+    (pin "1")
+    (pin "2")
+  )
+  (symbol (lib_id "Device:C") (at 157.48 82.55 0) (unit 1)
+    (in_bom yes) (on_board yes) (fields_autoplaced)
+    (property "Reference" "1µF" (id 0) (at 161.29 81.2799 0)
+      (effects (font (size 1.27 1.27)) (justify left))
+    )
+    (property "Value" "C" (id 1) (at 161.29 83.8199 0)
+      (effects (font (size 1.27 1.27)) (justify left))
+    )
+    (property "Footprint" "" (id 2) (at 158.4452 86.36 0)
+      (effects (font (size 1.27 1.27)) hide)
+    )
+    (property "Datasheet" "~" (id 3) (at 157.48 82.55 0)
+      (effects (font (size 1.27 1.27)) hide)
+    )
+    (pin "1")
+    (pin "2")
+  )
   (symbol (lib_id "power:GND") (at 210.82 95.25 90) (unit 1)
     (in_bom yes) (on_board yes) (fields_autoplaced)
@@
     )
     (property "Datasheet" "~" (id 3) (at 138.43 102.87 0)
-      (effects (font (size 1.27 1.27)) hide)
-    )
-    (pin "1")
-    (pin "2")
-  )
-  (symbol (lib_id "Device:C_Polarized") (at 157.48 82.55 0) (unit 1)
-    (in_bom yes) (on_board yes) (fields_autoplaced)
-    (property "Reference" "1µF?" (id 0) (at 161.29 80.3909 0)
-      (effects (font (size 1.27 1.27)) (justify left))
-    )
-    (property "Value" "C_Polarized" (id 1) (at 161.29 82.9309 0)
-      (effects (font (size 1.27 1.27)) (justify left))
-    )
-    (property "Footprint" "" (id 2) (at 158.4452 86.36 0)
-      (effects (font (size 1.27 1.27)) hide)
-    )
-    (property "Datasheet" "~" (id 3) (at 157.48 82.55 0)
       (effects (font (size 1.27 1.27)) hide)
     )
@@
     (pin "1")
   )
-  (symbol (lib_id "Device:C_Polarized") (at 157.48 102.87 0) (unit 1)
-    (in_bom yes) (on_board yes) (fields_autoplaced)
-    (property "Reference" "1µF?" (id 0) (at 161.29 100.7109 0)
-      (effects (font (size 1.27 1.27)) (justify left))
-    )
-    (property "Value" "C_Polarized" (id 1) (at 161.29 103.2509 0)
+  (symbol (lib_id "Device:C") (at 157.48 102.87 0) (unit 1)
+    (in_bom yes) (on_board yes) (fields_autoplaced)
+    (property "Reference" "1µF" (id 0) (at 161.29 101.5999 0)
+      (effects (font (size 1.27 1.27)) (justify left))
+    )
+    (property "Value" "C" (id 1) (at 161.29 104.1399 0)
       (effects (font (size 1.27 1.27)) (justify left))
     )
@@
     (pin "2")
   )
-  (symbol (lib_id "Device:C_Polarized") (at 190.5 102.87 0) (unit 1)
-    (in_bom yes) (on_board yes) (fields_autoplaced)
-    (property "Reference" "1µF?" (id 0) (at 194.31 100.7109 0)
-      (effects (font (size 1.27 1.27)) (justify left))
-    )
-    (property "Value" "C_Polarized" (id 1) (at 194.31 103.2509 0)
-      (effects (font (size 1.27 1.27)) (justify left))
-    )
+  (symbol (lib_id "Device:C") (at 190.5 102.87 0) (unit 1)
+    (in_bom yes) (on_board yes) (fields_autoplaced)
+    (property "Reference" "1µF" (id 0) (at 194.31 101.5999 0)
+      (effects (font (size 1.27 1.27)) (justify left))
+    )
+    (property "Value" "C" (id 1) (at 194.31 104.1399 0)
+      (effects (font (size 1.27 1.27)) (justify left))
+    )
